File: numpad_Schematics/numpad.kicad_sch (KiCad schematic)
At the start: 35 parts, among them U1 ESP32-DEVKIT-V1 Matrix Handler

Commit message: saving basic PCB design
Parts:
- removed SW1, SW10, SW11, SW12, SW13, SW14, SW15, SW16, SW17, SW2, SW3, SW4, SW5, SW6, SW7, SW8, SW9: ~, symbol tigmitSymbolLib:Switch_+_LED
- added J1: Encoder input, TIGMIT_KEYBOARD_FOOTPRINTS:PinHeader_1x05_P2.54mm_Vertical, symbol TIGMIT_KEBOARD_SYMBOLS:Conn_01x05_Pin
- added J2: power module input, TIGMIT_KEYBOARD_FOOTPRINTS:PinHeader_1x04_P2.54mm_Vertical, symbol TIGMIT_KEBOARD_SYMBOLS:Conn_01x04_Pin
- added J3: Display, TIGMIT_KEYBOARD_FOOTPRINTS:PinHeader_1x04_P2.54mm_Vertical, symbol TIGMIT_KEBOARD_SYMBOLS:Conn_01x04_Pin
- added R1, R2, R3, R4, R5: 10K, TIGMIT_KEYBOARD_FOOTPRINTS:R_Axial_DIN0204_L3.6mm_D1.6mm_P7.62mm_Horizontal, symbol TIGMIT_KEBOARD_SYMBOLS:Placeholder_Resistor
- added S1, S2, S3: MX_stab, TIGMIT_KEYBOARD_FOOTPRINTS:STAB_MX_2u, symbol TIGMIT_KEBOARD_SYMBOLS:MX_stab
- added SW1, SW10, SW11, SW12, SW13, SW14, SW15, SW16, SW17, SW2, SW3, SW4, SW5, SW6, SW7, SW8, SW9: ~, TIGMIT_KEYBOARD_FOOTPRINTS:hotswap socket with neopixel, symbol TIGMIT_KEBOARD_SYMBOLS:Switch_+_LED
- added U2: BOB-12009, TIGMIT_KEYBOARD_FOOTPRINTS:CONV_BOB-12009, symbol TIGMIT_KEBOARD_SYMBOLS:BOB-12009
- D1, D10, D11, D12, D13, D14, D15, D16, D17, D2, D3, D4, D5, D6, D7, D8, D9: footprint (none) -> TIGMIT_KEYBOARD_FOOTPRINTS:Diode_SOD-123
- U1: footprint tigmitLib:ESP32 Vroom Devkit V1 -> TIGMIT_KEYBOARD_FOOTPRINTS:ESP32 Vroom Devkit V1
Connections:
- net Row0 is gone; now on net Col2: U1.24 (D26)
- net Col0: now also D1.2 (A)
- net Col2: now also R1.1, SW1.1, SW2.1, SW3.1, SW4.1
- net Row1: now also R2.1, SW5.1, SW6.1, SW7.1
- net Row2: now also R3.1, SW10.1, SW11.1, SW8.1, SW9.1
- net Row3: now also R4.1, SW12.1, SW13.1, SW14.1
- net Row4: now also R5.1, SW15.1, SW16.1, SW17.1
- net at D14.1 (K): now also SW14.2
- net at D17.1 (K): now also SW17.2
- net at D8.1 (K): now also SW8.2
- net at D12.1 (K): now also SW12.2
- net at D11.1 (K): now also SW11.2
- net at D9.1 (K): now also SW9.2
- net at D7.1 (K): now also SW7.2
- net at D4.1 (K): now also SW4.2
- net at D15.1 (K): now also SW15.2
- net at D2.1 (K): now also SW2.2
- net at D5.1 (K): now also SW5.2
- net at D6.1 (K): now also SW6.2
- net at D10.1 (K): now also SW10.2
- net at D13.1 (K): now also SW13.2
- net at D16.1 (K): now also SW16.2
- net at D3.1 (K): now also SW3.2
- net at D1.1 (K): now also SW1.2
- net LV: now reaches U1.1 (3V3)
- net LV: now also J1.2 (Pin_2), J3.3 (Pin_3), U2.LV
- net NEOPIXEL_CONTROLL: now reaches U1.10 (D19)
- net NEOPIXEL_CONTROLL: now also U2.LV1
- net SDA: now reaches U1.11 (D21)
- net SDA: now also J3.1 (Pin_1)
- net SCL: now reaches U1.14 (D22)
- net SCL: now also J3.2 (Pin_2)
- net batt_voltage_Pin: now reaches U1.19 (D34)
- net batt_voltage_Pin: now also J2.2 (Pin_2)
- net GND: now reaches U1.2 (GND), U1.29 (GND)
- net GND: now also J1.1 (Pin_1), J2.3 (Pin_3), J3.4 (Pin_4), R1.2, R2.2, R3.2, R4.2, R5.2, SW1.6-GND (GND), SW10.6-GND (GND), SW11.6-GND (GND), SW12.6-GND (GND), SW13.6-GND (GND), SW14.6-GND (GND), SW15.6-GND (GND), SW16.6-GND (GND), SW17.6-GND (GND), SW2.6-GND (GND), SW3.6-GND (GND), SW4.6-GND (GND), SW5.6-GND (GND), SW6.6-GND (GND), SW7.6-GND (GND), SW8.6-GND (GND), SW9.6-GND (GND), U2.GND_1 (GND), U2.GND_2 (GND)
- net ENC_SW: now reaches U1.3 (D15)
- net ENC_SW: now also J1.3 (Pin_3)
- net HV: now reaches U1.30 (VIN)
- net HV: now also J2.4 (Pin_4), SW1.3-VDD (VDD), SW10.3-VDD (VDD), SW11.3-VDD (VDD), SW12.3-VDD (VDD), SW13.3-VDD (VDD), SW14.3-VDD (VDD), SW15.3-VDD (VDD), SW16.3-VDD (VDD), SW17.3-VDD (VDD), SW2.3-VDD (VDD), SW3.3-VDD (VDD), SW4.3-VDD (VDD), SW5.3-VDD (VDD), SW6.3-VDD (VDD), SW7.3-VDD (VDD), SW8.3-VDD (VDD), SW9.3-VDD (VDD), U2.HV
- net ENC_CLK: now reaches U1.4 (D2)
- net ENC_CLK: now also J1.5 (Pin_5)
- net ENC_DT: now reaches U1.5 (D4)
- net ENC_DT: now also J1.4 (Pin_4)
- net batt_chargesense: now reaches U1.8 (D5)
- net batt_chargesense: now also J2.1 (Pin_1)
- new net: SW4.4-DOUT (DO), SW5.5-DIN (DI)
- new net: SW3.4-DOUT (DO), SW4.5-DIN (DI)
- new net: SW12.4-DOUT (DO), SW13.5-DIN (DI)
- new net: SW11.4-DOUT (DO), SW12.5-DIN (DI)
- new net: SW2.4-DOUT (DO), SW3.5-DIN (DI)
- new net: SW1.4-DOUT (DO), SW2.5-DIN (DI)
- new net: SW16.4-DOUT (DO), SW17.5-DIN (DI)
- new net: SW5.4-DOUT (DO), SW6.5-DIN (DI)
- new net: SW14.4-DOUT (DO), SW15.5-DIN (DI)
- new net: SW13.4-DOUT (DO), SW14.5-DIN (DI)
- new net: SW10.4-DOUT (DO), SW11.5-DIN (DI)
- new net: SW10.5-DIN (DI), SW9.4-DOUT (DO)
- new net: SW15.4-DOUT (DO), SW16.5-DIN (DI)
- new net: SW7.4-DOUT (DO), SW8.5-DIN (DI)
- new net: SW6.4-DOUT (DO), SW7.5-DIN (DI)
- new net: SW8.4-DOUT (DO), SW9.5-DIN (DI)
- new net NEOPIXEL5VData: SW1.5-DIN (DI), U2.HV1
- no-connect marks 0 -> 10
Other:
- moved on the sheet: D1, D10, D11, D12, D13, D14, D15, D16, D17, D2, D3, D4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

Commit message: case and pcb design
Parts:
- removed J2: power module input, TIGMIT_KEYBOARD_FOOTPRINTS:PinHeader_1x04_P2.54mm_Vertical, symbol TIGMIT_KEBOARD_SYMBOLS:Conn_01x04_Pin
- removed S1, S2, S3: MX_stab, TIGMIT_KEYBOARD_FOOTPRINTS:STAB_MX_2u, symbol TIGMIT_KEBOARD_SYMBOLS:MX_stab
- removed U1: ESP32-DEVKIT-V1 Matrix Handler, TIGMIT_KEYBOARD_FOOTPRINTS:ESP32 Vroom Devkit V1, symbol ESP32-DEVKIT-V1:ESP32-DEVKIT-V1
- added C1: 10uF, Capacitor_Tantalum_SMD:CP_EIA-3528-12_Kemet-T, symbol TIGMIT_KEBOARD_SYMBOLS:C
- added C2: 0.1uF, Capacitor_Tantalum_SMD:CP_EIA-3528-12_Kemet-T, symbol TIGMIT_KEBOARD_SYMBOLS:C
- added C3: tbd, Capacitor_Tantalum_SMD:CP_EIA-3528-12_Kemet-T, symbol TIGMIT_KEBOARD_SYMBOLS:C
- added J2: pwr input, tigmitNIGHTLY:PinHeader_1x05_P2.54mm_Vertical, symbol TIGMIT_KEBOARD_SYMBOLS:Conn_01x05_Pin
- added J4: UART Download, Connector_PinHeader_2.54mm:PinHeader_1x03_P2.54mm_Horizontal, symbol TIGMIT_KEBOARD_SYMBOLS:Conn_01x03_Pin
- added R6: 10K, tigmitNIGHTLY:R_Axial_DIN0204_L3.6mm_D1.6mm_P7.62mm_Horizontal, symbol TIGMIT_KEBOARD_SYMBOLS:Placeholder_Resistor
- added SW18: SW_Push, tigmitNIGHTLY:tigmit pushbutton, symbol TIGMIT_KEBOARD_SYMBOLS:SW_Push
- added U3: ESP32-WROOM-32, tigmitNIGHTLY:ESP32-WROOM-32 tigmit, symbol TIGMIT_KEBOARD_SYMBOLS:ESP32-WROOM-32
- D1, D10, D11, D12, D13, D14, D15, D16, D17, D2, D3, D4, D5, D6, D7, D8, D9: footprint TIGMIT_KEYBOARD_FOOTPRINTS:Diode_SOD-123 -> tigmitNIGHTLY:Diode_SOD-123; symbol Device:D -> TIGMIT_KEBOARD_SYMBOLS:D
- J1: footprint TIGMIT_KEYBOARD_FOOTPRINTS:PinHeader_1x05_P2.54mm_Vertical -> tigmitNIGHTLY:PinHeader_1x05_P2.54mm_Vertical
- J3: footprint TIGMIT_KEYBOARD_FOOTPRINTS:PinHeader_1x04_P2.54mm_Vertical -> tigmitNIGHTLY:PinHeader_1x04_P2.54mm_Vertical
- R1, R2, R3, R4, R5: footprint TIGMIT_KEYBOARD_FOOTPRINTS:R_Axial_DIN0204_L3.6mm_D1.6mm_P7.62mm_Horizontal -> tigmitNIGHTLY:R_Axial_DIN0204_L3.6mm_D1.6mm_P7.62mm_Horizontal
- SW1, SW10, SW11, SW12, SW13, SW14, SW15, SW16, SW17, SW2, SW3, SW4, SW5, SW6, SW7, SW8, SW9: footprint TIGMIT_KEYBOARD_FOOTPRINTS:hotswap socket with neopixel -> tigmitNIGHTLY:hotswap socket with neopixel
- U2: footprint TIGMIT_KEYBOARD_FOOTPRINTS:CONV_BOB-12009 -> tigmitNIGHTLY:CONV_BOB-12009
Connections:
- net Col0: now also U3.11 (IO26)
- net Col1: now also U3.12 (IO27)
- net Col2: now also U3.13 (IO14); no longer R1.1, SW1.1, SW2.1, SW3.1, SW4.1
- net Col3: now also U3.14 (IO12)
- net ENC_CLK: now also U3.24 (IO2)
- net ENC_DT: now also U3.26 (IO4)
- net ENC_SW: now also U3.23 (IO15)
- net GND: now also J3.1 (Pin_1), C1.1, C2.1, C3.1, J2.1 (Pin_1), J4.1 (Pin_1), SW18.2, U3.1 (GND), U3.15 (GND), U3.38 (GND), U3.39 (GND); no longer J3.4 (Pin_4)
- net HV: now also J2.3 (Pin_3)
- net LV: now also J3.2 (Pin_2), C1.2, C2.2, J2.2 (Pin_2), R6.1, U3.2 (VDD); no longer J3.3 (Pin_3)
- net Row1: now also U3.7 (IO35)
- net Row2: now also U3.8 (IO32)
- net Row3: now also U3.9 (IO33)
- net Row4: now also U3.10 (IO25)
- net SCL: now also J3.3 (Pin_3), U3.36 (IO22); no longer J3.2 (Pin_2)
- net SDA: now also J3.4 (Pin_4), U3.33 (IO21); no longer J3.1 (Pin_1)
- net batt_chargesense: now also J2.4 (Pin_4), U3.29 (IO5)
- net batt_voltage_Pin: now also J2.5 (Pin_5), U3.16 (IO13)
- net NEOPIXEL5VData renamed NEOPIXEL5VData_KEYS
- net NEOPIXEL_CONTROLL renamed NEOPIXEL_CONTROLL_KEYS
- net NEOPIXEL_CONTROLL_KEYS: now also U3.31 (IO19)
- new net BOOT: SW18.1, U3.25 (IO0)
- new net ENable: C3.2, R6.2, U3.3 (EN)
- new net RXD0: J4.2 (Pin_2), U3.34 (RXD0/IO3)
- new net Row0: R1.1, SW1.1, SW2.1, SW3.1, SW4.1, U3.6 (IO34)
- new net TXD0: J4.3 (Pin_3), U3.35 (TXD0/IO1)
- no-connect marks 10 -> 17
Other:
- moved on the sheet: D1, D10, D11, D12, D13, D14, D15, D16, D17, D2, D3, D4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
